File: resources/schematics/main-board-multi/main-board/main-board.sch (KiCad schematic (older format))
At the start: 6 parts, among them J1 Conn_01x02_Female, J2 Conn_01x04_Female, J3 Conn_01x03_Female

Commit message: Refactor PCB - batch-20201231
Parts:
- removed J3: Conn_01x03_Female, Connector_PinSocket_2.54mm:PinSocket_1x03_P2.54mm_Vertical, symbol Connector:Conn_01x03_Female
- added J3: Conn_01x04_Female, digikey-footprints:PinHeader_1x4_P2.54mm_Drill1.02mm, symbol Connector:Conn_01x04_Female
- added R3, R4: 10K, Resistor_THT:R_Axial_DIN0309_L9.0mm_D3.2mm_P12.70mm_Horizontal, symbol Device:R
- added SW1: Switch_DPDT_7x7mm, symbol clvlabs-kicad-symbols:Switch_DPDT_7x7mm
- added SW2, SW3: SW_Push_45deg, Button_Switch_THT:SW_PUSH_6mm_H7.3mm, symbol Switch:SW_Push_45deg
- J1: footprint Connector_PinSocket_2.54mm:PinSocket_1x02_P2.54mm_Vertical -> digikey-footprints:PinHeader_1x2_P2.54mm_Drill1.02mm
- J2: footprint Connector_PinSocket_2.54mm:PinSocket_1x04_P2.54mm_Vertical -> digikey-footprints:PinHeader_1x4_P2.54mm_Drill1.02mm
Connections:
- net +5V: now also J2.1 (Pin_1), J3.4 (Pin_4), SW2.2, SW3.2; no longer J2.2 (Pin_2)
- net GND: now also J2.2 (Pin_2), J3.1 (Pin_1), R3.1, R4.1, SW1.2 (COM1); no longer J1.1 (Pin_1), J2.1 (Pin_1)
- net VIN: now also SW1.5 (COM2); no longer J1.2 (Pin_2)
- net PING_ECHO_PIN: now reaches A1.20 (A1)
- net PING_ECHO_PIN: now also J3.2 (Pin_2)
- net BUTTON_UP_PIN: now reaches A1.6 (D3)
- net BUTTON_UP_PIN: now also R3.2, SW2.1
- net BUTTON_DOWN_PIN: now reaches A1.7 (D4)
- net BUTTON_DOWN_PIN: now also R4.2, SW3.1
- net DISTANCE_SENSOR_PIN renamed PING_TRIGGER_PIN
- net PING_TRIGGER_PIN: now also J3.3 (Pin_3)
- new net BATT_GND: J1.1 (Pin_1), SW1.1 (NO1)
- new net BATT_VIN: J1.2 (Pin_2), SW1.4 (NO2)
Other:
- moved on the sheet: A1, J1, J2, R1, R2
